Commit message: refactoring folders

File: world_sim/urdf/robot.xacro (robot description, xacro)
@@ -68,6 +68,6 @@
     </xacro:scout_wheel_type2>
     <!-- Additional definitions -->
-    <xacro:include filename="$(find custom_world)/urdf/sensors.xacro" />
+    <xacro:include filename="$(find world_sim)/urdf/sensors.xacro" />
     <!-- Gazebo definitions  -->
-    <xacro:include filename="$(find custom_world)/urdf/robot_gazebo.xacro" />
+    <xacro:include filename="$(find world_sim)/urdf/robot_gazebo.xacro" />
 </robot>

File: world_sim/urdf/rplidar.xacro (robot description, xacro)
@@ -13,5 +13,5 @@
         <origin xyz="0 0 -0.03125" rpy="1.5707 0 0" />
         <geometry>
-          <mesh filename="package://custom_world/meshes/rplidar.dae" scale="0.001 0.001 0.001" />
+          <mesh filename="package://world_sim/meshes/rplidar.dae" scale="0.001 0.001 0.001" />
         </geometry>
       </visual>

File: world_sim/urdf/sensors.xacro (robot description, xacro)
@@ -3,6 +3,6 @@
   <!-- Includes -->
   <xacro:include filename="$(find realsense2_description)/urdf/_d435i.urdf.xacro" />
-  <xacro:include filename="$(find custom_world)/urdf/_d435.gazebo.xacro" />
-  <xacro:include filename="$(find custom_world)/urdf/rplidar.xacro" />
+  <xacro:include filename="$(find world_sim)/urdf/_d435.gazebo.xacro" />
+  <xacro:include filename="$(find world_sim)/urdf/rplidar.xacro" />
   <!-- Realsense sensor -->
   <xacro:sensor_d435i parent="base_link" use_nominal_extrinsics="true">
